File: wristband.kicad_sch (KiCad schematic)
At the start: 132 parts, among them J1 TC2030, J2 B4B-XH-A_LF__SN_, J3 USB_C_Receptacle, M1 Motor_DC, Q1 2N7002, Q2 FS8205, SW1 SW_Push, U1 BQ24075RGT, U10 CP2102N-Axx-xQFN20, U11 TPD4E05U06DQA, U12 DW01A, U13 MCP1640Bx-xCHY, U2 TS3USBCA410, U3 TPS62840DLCR, U4 DRV8876PWPT, U5 nRF52840, U6 AS5600, U7 MAX17048G_T10, U8 TPD4E05U06DQA, U9 SN74LVC2T45DCUR

Commit message: Add files via upload
Parts:
- removed D4: 1A, symbol Device:D_Schottky
- removed M1: Motor_DC, Connector_Wire:SolderWire-1x02_P1.27mm_D1.5mm, symbol Motor:Motor_DC
- removed U13: MCP1640Bx-xCHY, Package_TO_SOT_SMD:SOT-23-6, symbol Regulator_Switching:MCP1640Bx-xCHY
- added C50, C51, C52: 22uF, symbol Device:C
- added C53: 2.2uF, symbol Device:C
- added C54: 1nF, symbol Device:C
- added C55: 30pF, symbol Device:C
- added C56: 10uF, symbol Device:C
- added PS2: TPS61288LRQQR, TPS61288LRQQR:CONV_TPS61288LRQQR, symbol TPS61288LRQQR:TPS61288LRQQR
- C48: value 10u -> 0.1u
- C49: value 22u -> 0.1uF
- L4: value 4.7u -> 2.2uH
- R33: value 316k -> 36.5k
- R34: value 100k -> 36.5k
Connections:
- net +BATT: now also C56.1, PS2.7 (VIN)
- net 5V_ENC: no longer L4.1
- net GND: now also C50.2, C51.2, C52.2, C56.2; no longer C49.1, R34.2
- net MCU_GPIO: now also PS2.6 (EN)
- net VMOTOR: no longer C15.2, C17.2, C18.2, TP5.1, U4.11 (VM)
- net at R33.1: now also C54.2; no longer C49.2
- net at R34.1: now also C55.2; no longer R33.2
- new net: C54.1, C55.1, PS2.2 (COMP)
- new net: C49.1, L4.1, PS2.4 (SW), PS2.9 (SW__1)
- new net: C49.2, PS2.8 (BST)
- new net: C53.1, PS2.11 (VCC)
- new net 7V_MOTOR: C15.2, C17.2, C18.2, C50.1, C51.1, C52.1, PS2.5 (VOUT), TP5.1, U4.11 (VM)
- new net AGND: C53.2, PS2.10 (AGND), PS2.3 (PGND), R33.2, R34.2
Other:
- moved on the sheet: C21, C22, C23, C28, C29, C30, C31, C32, C33, C34, C35, C36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
